Commit message: urdf finalize, dynamics phase complete

File: resource/pogo/urdf/pogo.urdf (robot description, URDF)
Before this commit: robot pogo_test, 6 links, 5 joints
Links:
- added link head; visual sphere radius=0.15
- link foot: mass 0 -> None; geometry 
- link tip: geometry collision sphere radius=0.05; visual mesh filename=package://pogo_test/meshes/tip.STL
Joints:
- added joint mass_head: type fixed, parent mass, child head, origin xyz=0 0 1.26 rpy=0 0 0
