Commit message: pogo_1D urdf for tuning spring characteristics

File: resource/pogo/urdf/pogo_1D.urdf (robot description, URDF)
Before this commit: robot pogo, 7 links, 6 joints
Links:
- added link base
- added link world
Joints:
- added joint base_base_pogo: type prismatic, parent base, child base_pogo, origin xyz=0 0 0 rpy=0 0 0, axis 0 0 1, limit lower=0
- added joint base_world: type fixed, parent world, child base, origin xyz=0 0 0 rpy=0 0 0, axis 0 0 0
- joint base_cross: axis 0 1 0 -> 0 0 0; limit lower=-1.0472 upper=1.0472 effort=700 -> (none); type revolute -> fixed
- joint cross_guide: axis 1 0 0 -> 0 0 0; limit lower=-1.0472 upper=1.0472 effort=700 -> (none); type revolute -> fixed

Commit message: pogo characteristics fully determined

File: resource/pogo/urdf/pogo_1D.urdf (robot description, URDF)
Before this commit: robot pogo_test, 9 links, 8 joints
Joints:
- joint guide_mass: limit lower=0 upper=0.4 effort=3000 -> lower=0 upper=0.4 effort=3500
